Commit message: first commit

File: catkin_ws/src/multi_robot_scenario/xacro/p3dx/inertia_tensors.xacro (robot description, xacro)
@@ -34,4 +34,14 @@
     </inertial>
   </xacro:macro>
+    <xacro:macro name="our_trapezoid" params="x y z mass">
+    <inertial>
+      <origin xyz="0.0 0.0 -0.051054" rpy="0 0 0"/>
+      <mass value="${mass}" />
+      <inertia
+        ixx="0.000054" ixy="0.0" ixz="0.0"
+        iyy="0.000047" iyz="0.0"
+        izz="0.000010" />
+    </inertial>
+  </xacro:macro>
   <!-- #################### versions with origin #################### -->
   <xacro:macro name="sphere_inertial_with_origin" params="radius mass *origin">

File: catkin_ws/src/multi_robot_scenario/xacro/p3dx/pioneer3dx.xacro (robot description, xacro)
@@ -5,20 +5,17 @@
   <!-- Import robot -->
   <xacro:include filename="$(find multi_robot_scenario)/xacro/p3dx/pioneer3dx_body.xacro"/>
-  <xacro:pioneer3dx_body name="chassis" parent="base_link" meshes="package://gazebo_plugins/test/multi_robot_scenario/meshes/p3dx"/>
-  <!-- Laser -->
+  <xacro:pioneer3dx_body name="chassis" parent="base_link" meshes="package://multi_robot_scenario/meshes/p3dx"/>
+  <!-- uncomment 13 to 29 the below line to use other sensors like velodyne and hokuyo camera -->
+  <!--
   <xacro:include filename="$(find multi_robot_scenario)/xacro/laser/hokuyo.xacro"/>
   <xacro:laser name="front_laser" parent="chassis" xyz="0.125 0 0.25" rpy="0 0 0" meshes="package://gazebo_plugins/test/multi_robot_scenario/meshes/laser"/>
-  <!-- GPU Laser
-  <xacro:include filename="$(find multi_robot_scenario)/xacro/laser/hokuyo_gpu.xacro"/>
-  <xacro:laser_gpu name="front_laser" parent="chassis" xyz="0.16 0 0.1" rpy="0 0 0" meshes="package://gazebo_plugins/test/multi_robot_scenario/meshes/laser" />
-    -->
   <xacro:include filename="$(find multi_robot_scenario)/xacro/camera/camera.xacro"/>
   <xacro:cam name="front_camera" parent="chassis" xyz="0.025 0 0.32" rpy="0 0 0" />
   <xacro:include filename="$(find multi_robot_scenario)/xacro/camera/cameraD.xacro"/>
   <xacro:camD name="cameraD" parent="chassis" xyz="0.025 0 0.32" rpy="0 0 0" />
-  <!-- Velodyne -->
   <xacro:include filename="$(find velodyne_description)/urdf/VLP-16.urdf.xacro"/>
   <xacro:VLP-16 parent="base_link" name="velodyne" topic="/velodyne_points" hz="10" samples="360" gpu="false" min_angle="-1.57" max_angle="1.57" min_range="0.1">
     <origin xyz="0.125 0 0.25" rpy="0 0 0" />
   </xacro:VLP-16>
+-->
 </robot>

File: catkin_ws/src/multi_robot_scenario/xacro/p3dx/pioneer3dx_body.xacro (robot description, xacro)
@@ -3,26 +3,57 @@
   <xacro:include filename="inertia_tensors.xacro"/>
   <xacro:include filename="pioneer3dx_chassis.xacro"/>
-  <xacro:include filename="battery_block.xacro"/>
+  <xacro:include filename="pioneer3dx_chassis_2.xacro"/>
   <xacro:include filename="pioneer3dx_wheel.xacro"/>
-  <xacro:include filename="pioneer3dx_swivel.xacro"/>
-  <xacro:include filename="pioneer3dx_sonar.xacro"/>
+  <xacro:include filename="pioneer3dx_wheel_b.xacro"/>
   <xacro:include filename="pioneer3dx_plugins.xacro"/>
+  <xacro:include filename="$(find realsense2_description)/urdf/_d435.urdf.xacro"/>
   <xacro:macro name="pioneer3dx_body" params="name parent meshes">
-    <!-- base_link -->
     <link name="${parent}"/>
-    <!-- Chassis -->
-    <xacro:pioneer_chassis name="${name}" parent="base_link" xyz="0 0 0" rpy="0 0 0"  meshes="${meshes}"/>
-    <!-- Front Sonar -->
-    <xacro:pioneer_sonar name="sonar" parent="${name}" xyz="0.109 0 0.209" rpy="0 0 0"  meshes="${meshes}"/>
-    <!-- Akku0 -->
-    <xacro:battery_block name="battery0" parent="${name}" x="-0.14" y="0.00"  z="0.13" mass="2.5" />
-    <!-- Wheels -->
-    <xacro:pioneer_wheel side="right" parent="${name}"  xyz="0  0.15 0.09" rpy="0 0 0" radius="0.09" meshes="${meshes}"/>
-    <xacro:pioneer_wheel side="left"  parent="${name}"  xyz="0 -0.15 0.09" rpy="0 0 0" radius="0.09" meshes="${meshes}"/>
-    <xacro:pioneer_swivel parent="${name}"  xyz="-0.185 0 0.055" rpy="0 0 0" meshes="${meshes}"/>
-    <!-- Motor plugin -->
+    <xacro:pioneer_chassis name="${name}" parent="base_link" xyz="0 0 0" rpy="0 0 0" meshes="${meshes}"/>
+    <xacro:pioneer_chassis_2 name="${name}_2" parent="base_link" xyz="-0.2 0 0" rpy="0 0 0" meshes="${meshes}"/>
+    <xacro:pioneer_wheel side="right" parent="${name}" xyz="0 0.25 0" rpy="0 0 0" radius="0.125" meshes="${meshes}"/>
+    <xacro:pioneer_wheel side="left" parent="${name}" xyz="0 -0.25 0" rpy="0 0 0" radius="0.125" meshes="${meshes}"/>
+    <xacro:pioneer_wheel_b side="right_b" parent="${name}" xyz="-0.4 0.25 0" rpy="0 0 0" radius="0.125" meshes="${meshes}"/>
+    <xacro:pioneer_wheel_b side="left_b" parent="${name}" xyz="-0.4 -0.25 0" rpy="0 0 0" radius="0.125" meshes="${meshes}"/>
     <xacro:pioneer3dx_diff_drive />
-    <!-- Joints plugin -->
-    <xacro:pioneer3dx_joints_state_publisher />
-  </xacro:macro>
+    <xacro:pioneer3dx_joints_state_publisher /> <xacro:gazebo_control />
+    <xacro:sensor_d435 name="camera" topics_ns="realsense_camera" parent="base_link" publish_pointcloud="true">
+      <origin xyz="-0.3 -0.007 0.3" rpy="0 0 0" />
+    </xacro:sensor_d435>
+    <link name="imu_link">
+        <inertial>
+          <mass value="0.01"/>
+          <origin xyz="0 0 0.32" rpy="0 0 0"/>
+          <inertia ixx="1e-6" ixy="0" ixz="0" iyy="1e-6" iyz="0" izz="1e-6"/>
+        </inertial>
+        <visual>
+          <origin xyz="0 0 0" rpy="0 0 0"/>
+          <geometry>
+            <box size="0.01 0.01 0.01"/>
+          </geometry>
+        </visual>
+        <collision>
+          <origin xyz="0 0 0" rpy="0 0 0"/>
+          <geometry>
+            <box size="0.01 0.01 0.01"/>
+          </geometry>
+        </collision>
+      </link>
+      <joint name="imu_joint" type="fixed">
+        <parent link="base_link"/> <child link="imu_link"/>
+        <origin xyz="-0.37 -0.007 0.6" rpy="0 0 0"/>
+      </joint>
+      <gazebo reference="imu_link">
+        <gravity>true</gravity>
+        <sensor name="imu_sensor" type="imu">
+          <always_on>true</always_on>
+          <update_rate>100</update_rate> <visualize>true</visualize> <topic>__default_topic__</topic> <plugin filename="libgazebo_ros_imu_sensor.so" name="imu_plugin">
+            <topicName>imu/data</topicName> <bodyName>imu_link</bodyName> <updateRateHZ>100.0</updateRateHZ> <gaussianNoise>0.0</gaussianNoise> <xyzOffset>0 0 0</xyzOffset>
+            <rpyOffset>0 0 0</rpyOffset>
+            <frameName>imu_link</frameName> <initialOrientationAsReference>false</initialOrientationAsReference>
+          </plugin>
+          <pose>0 0 0 0 0 0</pose>
+        </sensor>
+    </gazebo>
+    </xacro:macro>
 </robot>

File: catkin_ws/src/multi_robot_scenario/xacro/p3dx/pioneer3dx_chassis.xacro (robot description, xacro)
@@ -11,5 +11,5 @@
   <link name="${name}">
     <visual name="chassis_visual">
-      <origin xyz="-0.045 0 0.148" rpy="0 0 0"/>
+      <origin xyz="${xyz}" rpy="${rpy}"/>
       <geometry name="pioneer_geom">
         <mesh filename="${meshes}/chassis.stl"/>
@@ -20,41 +20,19 @@
     </visual>
     <collision>
-      <origin xyz="-0.045 0 0.148" rpy="0 0 0"/>
+      <origin xyz="-0.045 0 0" rpy="0 0 0"/>
       <geometry>
         <mesh filename="${meshes}/chassis.stl"/>
       </geometry>
     </collision>
-    <xacro:box_inertial x="0.36" y="0.26"  z="0.18" mass="9.0" />
+    <xacro:cylinder_inertial length="0.255718" radius="0.01715" mass="6.0" />
+    <!-- <inertial>
+      <origin xyz="0 0 -0.034" rpy="0 0 0"/>
+      <mass value="9.0"/>
+      <inertia ixx="0.1" ixy="0.0" ixz="0.0" iyy="0.1" iyz="0.0" izz="0.1"/>
+    </inertial> -->
   </link>
   <gazebo reference="${name}">
     <material value="Gazebo/Red"/>
   </gazebo>
-  <!-- Top -->
-  <joint name="${name}_top_joint" type="fixed">
-    <origin xyz="-0.045 0 0.234" rpy="0 0 0"/>
-    <parent link="${name}"/>
-    <child link="top"/>
-  </joint>
-  <link name="top">
-    <visual>
-      <origin xyz="0 0 0" rpy="0 0 0"/>
-      <geometry name="top_geom">
-        <mesh filename="${meshes}/top.stl"/>
-      </geometry>
-      <material name="TopBlack">
-        <color rgba="0.038 0.038 0.038 1.0"/>
-      </material>
-    </visual>
-    <collision>
-    <origin xyz="0.0 0 0.0" rpy="0 0 0"/>
-      <geometry>
-        <mesh filename="${meshes}/top.stl"/>
-      </geometry>
-    </collision>
-    <xacro:box_inertial x="0.445" y="0.38"  z="0.01" mass="1.0" />
-  </link>
-  <gazebo reference="top">
-    <material value="Gazebo/Black"/>
-  </gazebo>
   </xacro:macro>
 </robot>

File: catkin_ws/src/multi_robot_scenario/xacro/p3dx/pioneer3dx_plugins.xacro (robot description, xacro)
@@ -3,33 +3,38 @@
   <xacro:macro name="pioneer3dx_joints_state_publisher">
     <gazebo>
-        <plugin name="joint_state_publisher" filename="libgazebo_ros_joint_state_publisher.so">
-          <robotNamespace></robotNamespace>
-          <jointName>chassis_swivel_joint, swivel_wheel_joint, left_hub_joint, right_hub_joint</jointName>
-          <updateRate>50.0</updateRate>
-          <alwaysOn>true</alwaysOn>
-        </plugin>
+      <plugin name="joint_state_publisher" filename="libgazebo_ros_joint_state_publisher.so">
+        <robotNamespace></robotNamespace>
+        <jointName>left_hub_joint, right_hub_joint</jointName>
+        <updateRate>50.0</updateRate>
+        <alwaysOn>true</alwaysOn>
+      </plugin>
     </gazebo>
   </xacro:macro>
   <xacro:macro name="pioneer3dx_diff_drive">
     <gazebo>
-        <plugin name="differential_drive_controller" filename="libgazebo_ros_diff_drive.so">
-            <rosDebugLevel>Debug</rosDebugLevel>
-            <robotNamespace></robotNamespace>
-            <publishWheelTF>false</publishWheelTF>
-            <publishWheelJointState>true</publishWheelJointState>
-            <alwaysOn>true</alwaysOn>
-            <leftJoint>left_hub_joint</leftJoint>
-            <rightJoint>right_hub_joint</rightJoint>
-            <wheelSeparation>0.3</wheelSeparation>
-            <wheelDiameter>0.18</wheelDiameter>
-            <wheelTorque>20</wheelTorque>
-            <wheelAcceleration>1.8</wheelAcceleration>
-            <commandTopic>cmd_vel</commandTopic>
-            <odometryTopic>odom</odometryTopic>
-            <odometryFrame>odom</odometryFrame>
-            <odometrySource>world</odometrySource>
-            <robotBaseFrame>base_link</robotBaseFrame>
-	    <updateRate>50</updateRate>
-        </plugin>
+      <plugin name="differential_drive_controller" filename="libgazebo_ros_diff_drive.so">
+        <rosDebugLevel>Debug</rosDebugLevel>
+        <robotNamespace></robotNamespace>
+        <publishWheelTF>false</publishWheelTF>
+        <publishWheelJointState>true</publishWheelJointState>
+        <alwaysOn>true</alwaysOn>
+        <leftJoint>left_hub_joint</leftJoint>
+        <rightJoint>right_hub_joint</rightJoint>
+        <wheelSeparation>0.3</wheelSeparation>
+        <wheelDiameter>0.18</wheelDiameter>
+        <wheelTorque>20</wheelTorque>
+        <wheelAcceleration>1.8</wheelAcceleration>
+        <commandTopic>cmd_vel</commandTopic>
+        <odometryTopic>odom</odometryTopic>
+        <odometryFrame>odom</odometryFrame>
+        <odometrySource>world</odometrySource> <robotBaseFrame>base_link</robotBaseFrame>
+        <updateRate>50</updateRate>
+      </plugin>
+    </gazebo>
+  </xacro:macro>
+  <xacro:macro name="gazebo_control">
+    <gazebo>
+      <plugin name="gazebo_ros_control" filename="libgazebo_ros_control.so">
+      </plugin>
     </gazebo>
   </xacro:macro>

File: catkin_ws/src/multi_robot_scenario/xacro/p3dx/pioneer3dx_wheel.xacro (robot description, xacro)
@@ -62,5 +62,5 @@
       <geometry>
         <!--<mesh filename="${meshes}/${side}_wheel.stl"/>-->
-        <cylinder radius="${radius}" length="0.01"/>
+        <cylinder radius="${radius}" length="0.1"/>
       </geometry>
     </collision>
